File: boards/radiva/radiva5.brd (EAGLE design)
At the start: 77.8 x 72.4 mm, 122 parts, among them CN1 BAT, IC1 TOUCH, IC10 VS1838, IC11 2.8V, IC12 1.8V, IC13 VS1053B, IC2 DC-DC 5V, IC3 TFT-DISPLAY-2.8, IC4 SY6280, IC5 ESP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

Commit message: fix bug on radiva5 brd
Routing:
- net +3V3: track 352.1 -> 356.7 mm
Changed lines of the file:
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@@
 <wire x1="60.6298" y1="29.4259" x2="60.6298" y2="28.2702" width="0.6096" layer="1"/>
 <wire x1="60.6298" y1="28.2702" x2="60.9854" y2="27.9146" width="0.6096" layer="1"/>
-<wire x1="72.9869" y1="28.5369" x2="72.9869" y2="31.4706" width="0.6096" layer="16"/>
+<wire x1="72.9869" y1="28.5369" x2="72.9869" y2="30.0482" width="0.6096" layer="16"/>
+<wire x1="72.9869" y1="30.0482" x2="72.9869" y2="31.4706" width="0.6096" layer="16"/>
 <wire x1="71.3867" y1="32.0929" x2="72.3646" y2="32.0929" width="0.4064" layer="16"/>
 <wire x1="72.3646" y1="32.0929" x2="72.9869" y2="31.4706" width="0.4064" layer="16"/>
@@
 <wire x1="73.2536" y1="8.001" x2="72.9869" y2="8.2677" width="0.6096" layer="16"/>
 <wire x1="72.9869" y1="8.2677" x2="72.9869" y2="14.4018" width="0.6096" layer="16"/>
-<wire x1="70.9422" y1="32.5374" x2="68.4971" y2="30.0923" width="0" layer="19" extent="16-16"/>
+<wire x1="68.4971" y1="30.0923" x2="72.9869" y2="30.0923" width="0.4064" layer="16"/>
+<wire x1="72.9869" y1="30.0923" x2="72.9869" y2="30.0482" width="0.4064" layer="16"/>
 </signal>
 <signal name="BAT+5V">

Commit message: little bug fix
Routing:
- net TFT_RST: track 115.5 -> 111.2 mm, vias 4 -> 3
Changed lines of the file:
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@@
 <grid distance="3.5" unitdist="mil" unit="mil" style="lines" multiple="1" display="yes" altdistance="1" altunitdist="mil" altunit="mil"/>
 <layers>
-<layer number="1" name="Top" color="4" fill="1" visible="no" active="yes"/>
+<layer number="1" name="Top" color="4" fill="1" visible="yes" active="yes"/>
 <layer number="2" name="Route2" color="1" fill="3" visible="no" active="no"/>
 <layer number="3" name="Route3" color="4" fill="3" visible="no" active="no"/>
@@
 <wire x1="43.9166" y1="50.1396" x2="44.0944" y2="50.4063" width="0.254" layer="16"/>
 <wire x1="44.0944" y1="50.4063" x2="44.8056" y2="50.4063" width="0.254" layer="16"/>
-<via x="58.0517" y="45.339" extent="1-16" drill="0.254" diameter="0.6096"/>
 <wire x1="64.8081" y1="26.2255" x2="67.1195" y2="26.2255" width="0.254" layer="16"/>
 <wire x1="64.8081" y1="32.893" x2="64.8081" y2="26.2255" width="0.254" layer="16"/>
@@
 <wire x1="46.5836" y1="42.5831" x2="46.8503" y2="42.8498" width="0.254" layer="16"/>
 <wire x1="46.8503" y1="42.8498" x2="47.5615" y2="42.8498" width="0.254" layer="16"/>
-<wire x1="58.0517" y1="45.339" x2="58.0517" y2="44.0055" width="0.254" layer="1"/>
-<wire x1="58.0517" y1="44.0055" x2="58.4073" y2="43.6499" width="0.254" layer="1"/>
-<wire x1="58.4073" y1="43.6499" x2="58.4073" y2="42.4053" width="0.254" layer="1"/>
-<wire x1="58.4073" y1="42.4053" x2="57.6072" y2="41.6052" width="0.254" layer="1"/>
 <wire x1="44.8056" y1="50.4063" x2="45.4279" y2="49.784" width="0.254" layer="16"/>
 <wire x1="45.4279" y1="49.784" x2="45.4279" y2="48.2727" width="0.254" layer="16"/>
